File: v2/schematics/tmp_adapter/teensy_adapter_v2/teensy_adapter.sch (EAGLE design)
At the start: 70 parts, among them IC1 TEENSY 3.6, IC2 ATMEGA1284P, IC3 MAX803REXR, IC4 DRV8835, IC5 L293D, J1 RADL, J10 RADL, J11 RADR, J12 Erw_PWM_1, J13 SWD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

Commit message: bugfix teensy adapter schematic: teensy pin 49/50 naming updated
Parts:
- C10: value 10n -> 10nF
- C11, C5, C6, C7, C9: value 1u -> 1uF
- C3, C4: value 220n -> 220nF
- C8: value 220u -> 220uF
- J1: value RADL -> RADL_SEL
- R29: value 5K -> 5k
- R30: value 100K -> 100k
Connections:
- net SERVO2_FB: now also IC1.49/A23; no longer IC1.49/A23/PWM
- net SERVO3_FB: now also IC1.50/A24; no longer IC1.50/A24/PWM
Other:
- note added: "Rev. 2.1"
- note removed: "Rev. 2.0"
Changed lines of the file:
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@@
 <?xml version="1.0" encoding="utf-8"?>
 <!DOCTYPE eagle SYSTEM "eagle.dtd">
-<eagle version="9.2.1">
+<eagle version="9.3.2">
 <drawing>
 <settings>
@@
 <part name="SUPPLY1" library="supply2_ts" deviceset="+5V" device="" value="+5V"/>
 <part name="GND1" library="supply1" library_urn="urn:adsk.eagle:library:371" deviceset="GND" device=""/>
-<part name="J1" library="pinhead_ts" deviceset="PINHD-1X3" device="" value="RADL"/>
+<part name="J1" library="pinhead_ts" deviceset="PINHD-1X3" device="" value="RADL_SEL"/>
 <part name="J2" library="pinhead_ts" deviceset="PINHD-1X4" device="" value="I2C_0"/>
 <part name="GND2" library="supply1" library_urn="urn:adsk.eagle:library:371" deviceset="GND" device=""/>
@@
 <part name="+3V8" library="supply1_ts" deviceset="+3V3" device=""/>
 <part name="GND8" library="supply1" library_urn="urn:adsk.eagle:library:371" deviceset="GND" device=""/>
-<part name="R29" library="rcl" deviceset="R-TRIMM" device="64W" value="5K"/>
+<part name="R29" library="rcl" deviceset="R-TRIMM" device="64W" value="5k"/>
 <part name="U4" library="user" deviceset="TPA3106D1" device=""/>
 <part name="GND14" library="supply1" deviceset="GND" device=""/>
 <part name="GND36" library="supply1" deviceset="GND" device=""/>
-<part name="R30" library="rcl" deviceset="R-EU_" device="0204/2V" value="100K"/>
-<part name="C11" library="rcl" deviceset="C-EU" device="025-025X050" value="1u"/>
-<part name="C10" library="rcl" deviceset="C-EU" device="025-025X050" value="10n"/>
-<part name="C4" library="rcl" deviceset="C-EU" device="025-025X050" value="220n"/>
-<part name="C3" library="rcl" deviceset="C-EU" device="025-025X050" value="220n"/>
-<part name="C9" library="rcl" deviceset="C-EU" device="025-025X050" value="1u"/>
-<part name="C6" library="rcl" deviceset="C-EU" device="025-025X050" value="1u"/>
-<part name="C5" library="rcl" deviceset="C-EU" device="025-025X050" value="1u"/>
+<part name="R30" library="rcl" deviceset="R-EU_" device="0204/2V" value="100k"/>
+<part name="C11" library="rcl" deviceset="C-EU" device="025-025X050" value="1uF"/>
+<part name="C10" library="rcl" deviceset="C-EU" device="025-025X050" value="10nF"/>
+<part name="C4" library="rcl" deviceset="C-EU" device="025-025X050" value="220nF"/>
+<part name="C3" library="rcl" deviceset="C-EU" device="025-025X050" value="220nF"/>
+<part name="C9" library="rcl" deviceset="C-EU" device="025-025X050" value="1uF"/>
+<part name="C6" library="rcl" deviceset="C-EU" device="025-025X050" value="1uF"/>
+<part name="C5" library="rcl" deviceset="C-EU" device="025-025X050" value="1uF"/>
 <part name="GND41" library="supply1" deviceset="GND" device=""/>
-<part name="C8" library="rcl" deviceset="CPOL-EU" device="E2.5-6" value="220u"/>
+<part name="C8" library="rcl" deviceset="CPOL-EU" device="E2.5-6" value="220uF"/>
 <part name="J14" library="pinhead_ts" deviceset="PINHD-1X2" device="" value="SPEAKER"/>
 <part name="IC4" library="pololu" deviceset="POLOLU_MOTOR_DRV8835" device="THROUGHHOLE" value="DRV8835"/>
@@
 <part name="IC5" library="st-microelectronics" deviceset="L293D" device="" package3d_urn="urn:adsk.eagle:package:26820/1"/>
 <part name="P+1" library="supply1" deviceset="V+" device="" value="+6V"/>
-<part name="C7" library="rcl" deviceset="C-EU" device="025-025X050" value="1u"/>
+<part name="C7" library="rcl" deviceset="C-EU" device="025-025X050" value="1uF"/>
 <part name="J15" library="pinhead_ts" deviceset="PINHD-1X2" device="" value="AUDIO"/>
 <part name="J16" library="pinhead_ts" deviceset="PINHD-1X3" device="" value="GAIN_0"/>
@@
 <text x="289.052" y="15.494" size="3.048" layer="94">c't-Bot Teensy 3.6
 Adapter Board v2</text>
-<text x="343.662" y="20.066" size="2.54" layer="94" font="vector">Rev. 2.0</text>
+<text x="343.662" y="20.066" size="2.54" layer="94" font="vector">Rev. 2.1</text>
 <text x="289.052" y="10.414" size="2.54" layer="94">CC BY-SA 4.0</text>
 </plain>
@@
 <instance part="C4" gate="G$1" x="43.434" y="68.58" smashed="yes" rot="MR0">
 <attribute name="NAME" x="41.91" y="68.961" size="1.778" layer="95" rot="MR0"/>
-<attribute name="VALUE" x="41.91" y="63.881" size="1.778" layer="96" rot="MR0"/>
+<attribute name="VALUE" x="43.18" y="63.881" size="1.778" layer="96" rot="MR0"/>
 </instance>
 <instance part="C3" gate="G$1" x="35.814" y="68.58" smashed="yes" rot="MR0">
 <attribute name="NAME" x="34.29" y="68.961" size="1.778" layer="95" rot="MR0"/>
-<attribute name="VALUE" x="34.29" y="63.881" size="1.778" layer="96" rot="MR0"/>
+<attribute name="VALUE" x="35.306" y="63.881" size="1.778" layer="96" rot="MR0"/>
 </instance>
 <instance part="C9" gate="G$1" x="40.894" y="30.48" smashed="yes" rot="MR0">
 <attribute name="NAME" x="39.37" y="30.861" size="1.778" layer="95" rot="MR0"/>
-<attribute name="VALUE" x="39.37" y="25.781" size="1.778" layer="96" rot="MR0"/>
+<attribute name="VALUE" x="40.132" y="25.781" size="1.778" layer="96" rot="MR0"/>
 </instance>
 <instance part="C6" gate="G$1" x="104.394" y="55.88" smashed="yes" rot="MR0">
@@
 <instance part="C8" gate="G$1" x="33.274" y="30.48" smashed="yes" rot="MR0">
 <attribute name="NAME" x="32.131" y="30.9626" size="1.778" layer="95" rot="MR0"/>
-<attribute name="VALUE" x="32.131" y="25.8826" size="1.778" layer="96" rot="MR0"/>
+<attribute name="VALUE" x="32.893" y="25.8826" size="1.778" layer="96" rot="MR0"/>
 </instance>
 <instance part="J14" gate="G$1" x="20.574" y="60.96" smashed="yes" rot="R180">
@@
 <net name="SERVO2_FB" class="0">
 <segment>
-<pinref part="IC1" gate="G$1" pin="49/A23/PWM"/>
+<pinref part="IC1" gate="G$1" pin="49/A23"/>
 <label x="279.654" y="132.08" size="1.778" layer="95"/>
 <wire x1="274.574" y1="132.08" x2="299.974" y2="132.08" width="0.1524" layer="91"/>
@@
 <net name="SERVO3_FB" class="0">
 <segment>
-<pinref part="IC1" gate="G$1" pin="50/A24/PWM"/>
+<pinref part="IC1" gate="G$1" pin="50/A24"/>
 <label x="279.654" y="134.62" size="1.778" layer="95"/>
 <wire x1="274.574" y1="134.62" x2="299.974" y2="134.62" width="0.1524" layer="91"/>
