File: v2/schematics/mainboard.sch (EAGLE design)
At the start: 161 parts, among them IC1 LM2596S-ADJ, IC10 TSOP34830, IC12 MAX803TEXR, IC2 LM2596S-5.0, IC3 LD1117A, IC4 DRV8835, IC5 LM393, IC6 TEENSY 3.6, IC7 PCF8574P, IC8 PCF8574P, IC9 UDN2981A, J1 Erw_Pow, J10 I2C_0, J11 I2C_3, J12 Uart_1, J13 Uart_6 (LP), J14 USB_Host, J15 BPS, J16 SPI0, J17 SPI_1, J18 SPI_2, J19 Erw_analog, J2 H-Bridge Mode, J20 Erw_GPIO, J21 Erw_PWM, J23 Erw_ENA, J24 ESP01 Prog, J25 Bat_In, J26 SWD, J27 SPEAKER, J28 AUDIO, J29 GAIN_0, J3 Servo_1, J30 GAIN_1, J31 SWD_KL02, J32 SWD_KL02, J33 Erw_Servo, J4 Servo_2, J5 Servo_3, J6 I2C_1, J7 BNO055, J8 Uart_2, J9 I2C0_5V, SW1 TL32PO, T1 BC547, U1 IRL3103, U3 BSS138, U4 BSS138, U6 TPA3106D1, X1 U0 max. 18V (!)

Commit message: ct-bot v2 schematic updated
 - bugfix for library references, non-managed libraries added as dedicated library (ct-bot.lbr)
 - wrong footprints reverted
 - bufix for wrong signals for servo supplies
 - bugfix reverse polarity protection
 - bugifx for line sensor voltage levels
 - small smd parts exchanged with TH alternatives (bs108, mcp101) (untested)
 - distance and transport box sensors updated with I2C (untested)
 - led driver updated for up to 25 mA per channel (untested)
 - audio amp switched to pam8403 (untested)
 - bugfix for ESP12 programming mode (circuit still incomplete)
 - missing signals on RPi interface header restored
 - spi header for additional channels added due to pin mapping sheet changes
 - missing header for uart5 added
 - several layout improvements
Parts:
- removed C29, C31: 6.8nF, rcl:C-EU025-025X050
- removed C30: 2.2nF, rcl:C-EU025-025X050
- removed ESP-01: WIRELESS-WIFI-ESP-01, DIYmodules-general:WIRELESS-WIFI-ESP-01
- removed IC12: MAX803TEXR, EAGLE-maxim-10:MAX803TEXR
- removed J33: Erw_Servo, DIYmodules-pinhead:PINHD-1X2
- removed R53, R54: 4k7, rcl:R-EU_0204/2V
- removed R55, R56: 10k, rcl:R-EU_0204/2V
- removed T1: BC547, transistor:BC547
- added D4: SB 540, diode:SCHOTTKY-DIODEDO201T15
- added IC11: UDN2981A, ct-bot:UDN2981A
- added IC13: PAM8403, ct-bot:PAM8403
- added J133: USB_Host, ct-bot:PINHD-1X4
- added J22: Erw_PWM, ct-bot:PINHD-1X6
- added R38: 220, rcl:R-EU_0204/2V
- added R39: 590, rcl:R-EU_0204/2V
- added R40: 115, rcl:R-EU_0204/2V
- added R41: 1k8, rcl:R-EU_0204/2V
- added R42: 4k7, rcl:R-EU_0204/2V
- added U2, U5, U7: BS108, ct-bot:BS108
- BT1: device SparkFun-Batteries:BATTERY-20MM_PTH -> ct-bot:BATTERY-20MM_PTH
- C11, C14: value 100nF -> 2.2nF
- C12, C15: value 100nF -> 6.8nF
- C13, C18: value 220uF -> 100nF; device rcl:CPOL-EUE5-10.5 -> rcl:C-EU025-025X050
- C16: value 100uF -> 100nF; device rcl:CPOL-EUE5-10.5 -> rcl:C-EU025-025X050
- C17: value 100nF -> 220uF; device rcl:C-EU025-025X050 -> rcl:CPOL-EUE2-5
- C19, C25: value 1u -> 100nF
- C20: value 10n -> 100uF; device rcl:C-EU025-025X050 -> rcl:CPOL-EUE2-5
- C21: value 220n -> 100nF
- C22: value 220n -> 470nF
- C23, C24, C27: value 1u -> 1uF
- C26: value 220u -> 470nF; device rcl:CPOL-EUE5-10.5 -> rcl:C-EU025-025X050
- C28: value 2.2nF -> 470uF; device rcl:C-EU025-025X050 -> rcl:CPOL-EUE3.5-8
- C3: value 1nF -> 220u; device rcl:C-EU025-025X050 -> rcl:CPOL-EUE5-10.5
- C4: value 220u -> 1nF; device rcl:CPOL-EUE5-10.5 -> rcl:C-EU025-025X050
- C9: device rcl:CPOL-EUE5-10.5 -> rcl:CPOL-EUE2-5
- D1, D2: value SB 540 -> 1N4148; device diode:SCHOTTKY-DIODEDO201T15 -> ct-bot:1N41480207/2V
- D3: value BAV99 -> SB 540; device diode:BAV199 -> diode:SCHOTTKY-DIODEDO201T15
- IC1, IC2: device linear:LM2596S -> ct-bot:LM2596S
- IC10: value TSOP34830 -> PCF8574P; device vishay-1:TSOP34830 -> ct-bot:PCF8574P
- IC3: device LD1117:LD1117 -> ct-bot:LD1117
- IC4: value DRV8835 -> LM393; device pololu:POLOLU_MOTOR_DRV8835THROUGHHOLE -> linear:LM393N; SPICEPREFIX (none) -> J
- IC5: value LM393 -> MCP101-300; device linear:LM393N -> ct-bot:MCP101; SPICEPREFIX J -> (none)
- IC6: value TEENSY 3.6 -> TSOP34830; device Teensy_3_6:TEENSY3_6--ALLPINS -> ct-bot:TSOP34830
- IC7: value PCF8574P -> DRV8835; device micro-philips:PCF8574P -> ct-bot:DRV8835THROUGHHOLE
- IC8: value PCF8574P -> TEENSY 3.6; device micro-philips:PCF8574P -> ct-bot:TEENSY3_6
- IC9: value UDN2981A -> PCA9634; device uln-udn:UDN2981A -> ct-bot:PCA9634-SO20
- J1: value Erw_Pow -> Bat_In; device DIYmodules-pinhead:PINHD-1X4 -> ct-bot:PINHD-1X2
- J10: value I2C_0 -> SPI_2; device DIYmodules-pinhead:PINHD-1X4 -> ct-bot:PINHD-1X6
- J11: value I2C_3 -> I2C_0; device DIYmodules-pinhead:PINHD-1X4 -> ct-bot:PINHD-1X4
- J12: value Uart_1 -> I2C_1; device DIYmodules-pinhead:PINHD-1X4 -> ct-bot:PINHD-1X4
- J13: value Uart_6 (LP) -> I2C_3; device DIYmodules-pinhead:PINHD-1X4 -> ct-bot:PINHD-1X4
- J14: value USB_Host -> BNO055; device DIYmodules-pinhead:PINHD-1X4 -> ct-bot:PINHD-1X6
- J15: value BPS -> Uart_2; device DIYmodules-pinhead:PINHD-1X3 -> ct-bot:PINHD-1X4
- J16: value SPI0 -> Uart_5; device DIYmodules-pinhead:PINHD-1X8 -> ct-bot:PINHD-1X4
- J17: value SPI_1 -> Uart_6 (LP); device DIYmodules-pinhead:PINHD-1X6 -> ct-bot:PINHD-1X4
- J18: value SPI_2 -> BPS; device DIYmodules-pinhead:PINHD-1X7 -> ct-bot:PINHD-1X3
- J19: value Erw_analog -> Servo_2; device DIYmodules-pinhead:PINHD-1X2 -> ct-bot:PINHD-1X4
- J2: value H-Bridge Mode -> Erw_Pow; device DIYmodules-pinhead:PINHD-1X2 -> ct-bot:PINHD-1X4
- J20: value Erw_GPIO -> Servo_3; device DIYmodules-pinhead:PINHD-1X2 -> ct-bot:PINHD-1X4
- J21: value Erw_PWM -> Erw_Servo; device DIYmodules-pinhead:PINHD-1X6 -> ct-bot:PINHD-1X2
- J23: value Erw_ENA -> ESP01 Prog; device DIYmodules-pinhead:PINHD-1X8 -> ct-bot:PINHD-1X4
- J24: value ESP01 Prog -> SWD; device DIYmodules-pinhead:PINHD-1X3 -> ct-bot:PINHD-1X6
- J25: value Bat_In -> SWD_KL02; device DIYmodules-pinhead:PINHD-1X2 -> ct-bot:PINHD90-1X2/90
- J26: value SWD -> SWD_KL02; device DIYmodules-pinhead:PINHD-1X6 -> ct-bot:PINHD-1X2
- J27: value SPEAKER -> SPEAKER_L; device DIYmodules-pinhead:PINHD-1X2 -> ct-bot:PINHD-1X2
- J28: value AUDIO -> SPEAKER_R; device DIYmodules-pinhead:PINHD-1X2 -> ct-bot:PINHD-1X2
- J29: value GAIN_0 -> AUDIO_TEENSY; device DIYmodules-pinhead:PINHD-1X3 -> ct-bot:PINHD-1X3
- J3: device DIYmodules-pinhead:PINHD-1X4 -> ct-bot:PINHD-1X4
- J30: value GAIN_1 -> Erw_ENA; device DIYmodules-pinhead:PINHD-1X3 -> pinhead:PINHD-2X4
- J31: value SWD_KL02 -> Erw_GPIO; device DIYmodules-pinhead:PINHD-1X2 -> ct-bot:PINHD-1X2
- J32: value SWD_KL02 -> Erw_analog; device DIYmodules-pinhead:PINHD-1X2 -> ct-bot:PINHD-1X2
- J4: value Servo_2 -> H-Bridge Mode; device DIYmodules-pinhead:PINHD-1X4 -> ct-bot:PINHD-1X2
- J5: value Servo_3 -> I2C0_5V; device DIYmodules-pinhead:PINHD-1X4 -> ct-bot:PINHD-1X4
- J6: value I2C_1 -> SPI_0; device DIYmodules-pinhead:PINHD-1X4 -> con-harting-ml:ML10
- J7: value BNO055 -> SPI_0; device DIYmodules-pinhead:PINHD-1X6 -> ct-bot:PINHD-1X7
- J8: value Uart_2 -> SPI_0; device DIYmodules-pinhead:PINHD-1X4 -> ct-bot:PINHD-1X6
- J9: value I2C0_5V -> SPI_2; device DIYmodules-pinhead:PINHD-1X4 -> ct-bot:PINHD-1X7
- L1, L2: device inductors:09HCP -> ct-bot:INDUCTOR_09HCP
- LDR1, LDR2: device Seeed-Sensor:PHOTORESISTOR-5528-10K(2P-5.0X4.2MM) -> ct-bot:MPY54C569
- LED10, LED4: value blau -> rot
- LED11: value weiss -> blau
- LED12, LED6: value rot -> blau
- LED5: value blau -> weiss
- LED7: value orange -> gruen
- LED9: value gruen -> orange
- R1: value 100k -> 1k
- R10: value 100 -> 47k
- R11: value 10k -> 47k
- R12, R13: value 470k -> 210
- R14: value 5k -> 180; device rcl:R-TRIMM64W -> rcl:R-EU_0204/2V
- R15, R19: value 10k -> 180
- R16: value 1M -> 47k
- R17: value 10k -> 47k; device rcl:R-EU_0204/7 -> rcl:R-EU_0204/2V
- R18: value 15k -> 180
- R2: value 3k9 0.1% -> 100k
- R20: device rcl:R-TRIMM64W -> ct-bot:R-TRIMM64W
- R24: value 15k -> 10k
- R25: value 10k -> 15k
- R26: value 100k -> 5k; device rcl:R-EU_0204/2V -> ct-bot:R-TRIMM64W
- R27, R29, R46: value 4k7 -> 10k
- R28: value 4k7 -> 1M
- R3: value 1k 0.1% -> 22k
- R30: value 210 -> 10k
- R31: value 210 -> 15k
- R32, R33: value 180 -> 470k
- R34: value 47k -> 4k7
- R35: value 47k -> 100
- R36: value 100 -> 4k7
- R37: value 5k -> 3k9; device rcl:R-TRIMM64W -> rcl:R-EU_0204/2V
- R4: value 390 -> 100k
- R43: value 100k -> 4k7
- R44: value 180k -> 4k7
- R47: value 1k8 -> 10k
- R48: value 115 -> 4k7
- R49: value 590 -> 4k7
- R5: value 330 -> 3k9 0.1%
- R50: value 220 -> 5k; device rcl:R-EU_0204/2V -> ct-bot:R-TRIMM64W
- R51: value 3k9 -> ?
- R52: value 4k7 -> ?
- R6: value 120 -> 1k 0.1%
- R7: value 1k -> 390
- R8: value 100k -> 330
- R9: value 22k -> 120
- ST1: value Motor L -> Sensoren L; device DIYmodules-pinhead:PINHD-1X2 -> ct-bot:PS25-10PS25-10
- ST2: value Motor R -> Sensoren R; device DIYmodules-pinhead:PINHD-1X2 -> ct-bot:PS25-10PS25-10
- ST3: value Sensoren L -> Liniensensoren; device DIYmodules-pinhead:PINHD-1X10 -> ct-bot:PS25-5PS25-5
- ST4: value Sensoren R -> Motor R; device DIYmodules-pinhead:PINHD-1X10 -> ct-bot:PINHD90-1X2/90
- ST5: value RPI_Interface -> Motor L; device con-harting-ml:ML26 -> ct-bot:PINHD90-1X2/90
- ST6: value Maussensor -> RPI_Interface; device DIYmodules-pinhead:PINHD-1X10 -> con-harting-ml:ML26
- U3, U4: value BSS138 -> BS108; device DIYmodules-m-pad-2.1:BSS138 -> ct-bot:BS108
- U6: value TPA3106D1 -> BS108; device user:TPA3106D1 -> ct-bot:BS108
- X1: value U0 max. 18V (!) -> max. 18V; device con-ptr500:AK500/2-H -> ct-bot:SCHRAUBKLEMME/2
Connections:
- removed net DRV_ABSTAND: ST3.3, ST4.3
- removed net ESP_GPIO0: ESP-01.GPIO0, ESP-12.GPIO0, J24.2
- removed net ESP_GPIO2: ESP-01.GPIO2, ESP-12.GPIO2, J24.1
- removed net GAIN0: J29.2, U6.GAIN0
- removed net GAIN1: J30.2, U6.GAIN1
- removed net GPIO24: IC6.24, J20.1
- removed net INN: C24.1, U6.INN
- removed net INP: C25.1, U6.INP
- removed net LED_MCU: IC6.13/LED/ALT-PWM/SCK0, R11.1
- removed net LINE_IN: J28.2, R37.E
- removed net N$163: C25.2, R37.S
- removed net N$57: ST3.8, ST4.8
- removed net N$90: U6.FAULT, U6.MUTE
- removed net OUTN: C21.2, J27.1, U6.OUTN0, U6.OUTN1
- removed net OUTP: C22.2, J27.2, U6.OUTP0, U6.OUTP1
- removed net PWR_SERVO: J4.2, J5.2, ST5.22
- removed net ROSC: R26.2, U6.ROSC
- removed net SCHRANKE: R43.1, ST3.9
- removed net SCHRANKE_3V3: IC6.46/SCK2, J20.2, R43.2, R44.1
- removed net VBYP: C19.1, U6.VBYP
- removed net VREG: C20.1, J29.1, J30.1, U6.MSTR/SLV, U6.VREG
- new net ABST_SHUT_L: IC10.P3, U2.G
- new net ABST_SHUT_R: IC10.P4, U3.G
- new net GPIO_24: IC8.24, J31.1
- new net GPIO_46: IC8.46/SCK2, J31.2
- new net LINE_IN_L: J29.2, R50.A
- new net LINE_IN_R: C26.2, J29.3
- new net N$34: C10.1, R20.S, R21.1
- new net N$36: C13.1, R26.S, R27.1
- new net N$37: IC4B.+IN, R27.2, R28.1
- new net N$40: IC13.INL, R51.1
- new net N$41: C22.1, R51.2
- new net N$42: C22.2, R50.S
- new net N$43: IC13.-OUT_R, J28.1
- new net N$44: IC13.+OUT_R, J28.2
- new net N$46: IC13.INR, R52.1
- new net N$48: C26.1, R52.2
- new net RPI_3V3: ST6.11
- new net RPI_SPI0_CE1: ST6.10
- new net SERVO3_FB: ST6.14
- new net TEENSY_LED: IC8.13/LED/ALT-PWM/SCK0, U5.G
- new net VL53L0X_SHUT_L: ST1.4, U2.D
- new net VL53L0X_SHUT_R: ST2.4, U3.D
- net +3V3: now also C21.1, D1.C, IC4P.V+, IC6.VS, J18.3, J2.1, J23.1, J6.10, R11.1, R16.2, R17.2, R23.2, R26.E, R31.2, R32.2, R33.2, R35.2, R44.2, R45.2, R48.2, R49.2, R9.2, ST6.1, U6.G, U7.G; no longer C17.1, D3.C, ESP-01.CH_PD, ESP-01.VCC, IC10.VS, J1.1, J15.3, R12.2, R13.2, R14.E, R18.2, R19.2, R24.2, R27.2, R28.2, R35.1, R53.2, R54.2, R6.2, ST5.1, U3.G, U4.G
- net +5V: now also C16.1, C17.+, C18.1, C19.1, C20.+, C23.1, C24.1, C27.1, C28.+, IC10.A0, IC10.VDD, IC11.VS, IC13.PVDD, IC13.PVDD1, IC13.VDD, IC7.VCC, IC8.VIN, IC9.A0, IC9.A2, IC9.A4, IC9.VDD, J133.1, J15.2, J16.2, J2.2, J4.1, J5.2, J6.1, J8.1, R37.1, R38.1, R39.1, R40.1, R41.1, R42.1, R43.1, R46.2, R47.2, R8.2, ST1.3, ST2.3, ST6.23, ST6.25; no longer C12.1, C13.+, C14.1, C15.1, C16.+, C18.+, C32.1, IC4.VCC, IC5P.V+, IC6.VIN, IC7.VDD, IC8.A0, IC8.VDD, IC9.VS, J1.2, J16.1, J18.2, J2.1, J6.2, J8.2, R45.1, R46.1, R47.1, R48.1, R49.1, R5.2, R50.1, R51.1, R52.1, R55.2, R56.2, ST5.23, ST5.25, ST6.1
- net +6V: now also C3.+, C4.1, IC7.VIN, J19.2, J2.3, J20.2, R5.2, R7.1, ST6.22; no longer C3.1, C4.+, IC4.VIN, J1.3, R2.2, R4.1
- net 3V3_TEENSY: now also C32.1, IC5.VDD, IC8.3V3, J24.1; no longer IC12.VCC, IC6.3V3, J26.1
- net A22_DAC1: now also IC8.DAC1, J32.1; no longer IC6.DAC1, J19.1
- net AUDIO_OUT: now also IC8.DAC0, J29.1, J32.2; no longer IC6.DAC0, J19.2, J28.1
- net BAT+: now also X1-2.KL; no longer R1.2, X1-1.KL
- net BAT-: now also X1-1.KL; no longer X1-2.KL
- net BAT_IN: now also J1.1, R2.2, R4.2; no longer C26.+, C27.1, J25.1, R8.2, U6.!SHUTDOWN, U6.AVCC, U6.PVCC0, U6.PVCC1, U6.PVCC2, U6.PVCC3
- net BAT_IN_FB: now also IC8.39/A20/ALT-MISO0, R1.1; no longer IC6.39/A20/ALT-MISO0, R7.1
- net BPS: now also IC8.42, J18.1; no longer IC6.42, J15.1
- net DRV_ERW_1: now also IC11.O5, J30.2; no longer IC9.O4, J23.2
- net DRV_ERW_2: now also IC11.O6, J30.4; no longer IC9.O5, J23.4
- net DRV_ERW_3: now also IC11.O7, J30.6; no longer IC9.O6, J23.6
- net DRV_ERW_4: now also IC11.O8, J30.8; no longer IC9.O7, J23.8
- net DRV_KANTLED: now also IC11.O2, R14.2, R15.1; no longer IC9.O2, R32.2, R33.1
- net DRV_LINIE: now also IC11.O3, R18.2, R19.2; no longer IC9.O3, ST6.9
- net DRV_RADLED: now also IC11.O1, R12.2, R13.1; no longer IC9.O1, R30.2, R31.1
- net DRV_SCHRANKE: now also IC11.O4, ST1.9; no longer IC9.O8, ST3.7
- net ENA_ERW_1: now also IC10.P6, IC11.I5, J30.1; no longer IC8.P3, IC9.I4, J23.1
- net ENA_ERW_2: now also IC10.P7, IC11.I6, J30.3; no longer IC8.P4, IC9.I5, J23.3
- net ENA_ERW_3: now also IC11.I8, J30.5; no longer IC8.P5, IC9.I6, J23.5
- net ENA_ERW_4: now also IC11.I7, J30.7; no longer IC8.P6, IC9.I7, J23.7
- net ENA_KANTLED: now also IC10.P1, IC11.I2; no longer IC8.P1, IC9.I2
- net ENA_LINIE: now also IC10.P2, IC11.I3; no longer IC8.P2, IC9.I3
- net ENA_RADLED: now also IC10.P0, IC11.I1; no longer IC8.P0, IC9.I1
- net ENA_SCHRANKE: now also IC10.P5, IC11.I4; no longer IC8.P7, IC9.I8
- net ENC_L: now also R24.2, R25.1, ST1.1; no longer R17.2, R18.1, ST3.1
- net ENC_R: now also R30.2, R31.1, ST2.1; no longer R23.2, R24.1, ST4.1
- net FERNBED: now also IC6.OUT, IC8.28/ALT-MOSI0; no longer IC10.OUT, IC6.28/ALT-MOSI0
- net GND: now also C13.2, C16.2, C17.-, C18.2, C20.-, C21.2, C25.2, C28.-, C3.-, D4.A, IC10.A1, IC10.A2, IC10.VSS, IC11.GND, IC13.GND, IC13.PGND, IC13.PGND1, IC4P.V-, IC5.VSS, IC7.LGND, IC7.MGND, IC8.AGND, IC8.GND, IC9.A1, IC9.A3, IC9.A5, IC9.A6, IC9.OE, IC9.VSS, J1.2, J133.4, J14.3, J15.1, J16.1, J18.2, J19.1, J2.4, J20.1, J23.4, J6.2, J7.2, J8.2, R26.A, R50.E, R6.1, ST1.10, ST2.10, ST3.5, ST6.24, ST6.26, U2.S, U3.S, U4.S, U5.S; no longer C13.-, C16.-, C17.2, C18.-, C20.2, C26.-, C28.2, C29.2, C30.2, C31.2, C4.-, D1.A, ESP-01.GND, IC10.GND, IC12.GND, IC4.LGND, IC4.MGND, IC5P.V-, IC6.AGND, IC7.A0, IC7.A1, IC7.A2, IC7.VSS, IC8.A1, IC8.A2, IC8.VSS, IC9.GND, J1.4, J14.4, J15.2, J16.2, J18.1, J25.2, J26.3, J29.3, J30.3, J4.1, J6.1, J7.3, J8.1, R14.A, R26.1, R37.A, R44.2, R9.1, ST3.10, ST4.10, ST5.24, ST5.26, ST6.10, T1.E, U6.AGND0, U6.AGND1, U6.AGND2, U6.PAD, U6.PGND0, U6.PGND1, U6.PGND2, U6.PGND3
- net KANTE_L: now also IC8.18/A4/PWM/T/SDA0, R10.1, ST1.6; no longer IC6.18/A4/PWM/T/SDA0, R34.1, ST3.6
- net KANTE_R: now also IC8.19/A5/PWM/T/SCL0, R11.2, ST2.6; no longer IC6.19/A5/PWM/T/SCL0, R35.2, ST4.6
- net KL02_DC: now also J25.1, J26.1; no longer J31.1, J32.1
- net KL02_DD: now also J25.2, J26.2; no longer J31.2, J32.2
- net LDR_L: now also IC8.49/A23, R32.1; no longer IC6.49/A23/PWM, R13.1
- net LDR_R: now also IC8.50/A24, R33.1; no longer IC6.50/A24/PWM, R12.1
- net LINIE_L: now also IC8.A10, R17.1, ST3.3; no longer IC6.A10, ST6.7
- net LINIE_R: now also IC8.A11, R16.1, ST3.4; no longer IC6.A11, ST6.8
- net MOT_L_1: now also IC7.AOUT1, ST5.1; no longer IC4.AOUT1, ST1.1
- net MOT_L_2: now also IC7.AOUT2, ST5.2; no longer IC4.AOUT2, ST1.2
- net MOT_L_DIR: now also IC7.APHASE, IC8.40; no longer IC4.APHASE, IC6.40
- net MOT_L_PWM: now also IC7.AENBL, IC8.35/A16/PWM; no longer IC4.AENBL, IC6.35/A16/PWM
- net MOT_R_1: now also IC7.BOUT1, ST4.1; no longer IC4.BOUT1, ST2.1
- net MOT_R_2: now also IC7.BOUT2, ST4.2; no longer IC4.BOUT2, ST2.2
- net MOT_R_DIR: now also IC7.BPHASE, IC8.41; no longer IC4.BPHASE, IC6.41
- net MOT_R_PWM: now also IC7.BENBL, IC8.36/A17/PWM; no longer IC4.BENBL, IC6.36/A17/PWM
- net N$1: now also R18.1, ST3.2; no longer R36.2, ST4.7
- net N$10: now also IC4B.-IN, R30.1; no longer IC5A.+IN, R15.2, R16.1
- net N$11: now also R8.1; no longer R5.1
- net N$12: now also ESP-12.GPIO15, J23.3; no longer IC5B.+IN, R21.2, R22.1
- net N$13: now also IC9.LED2, LED10.C; no longer IC7.P2, LED6.C
- net N$14: now also ESP-12.GPIO0, J23.2; no longer IC5B.-IN, R23.1
- net N$15: now also IC9.LED3, LED9.C; no longer IC7.P3, LED7.C
- net N$16: now also IC9.LED4; no longer IC7.P4
- net N$17: now also IC9.LED5, LED7.C; no longer IC7.P5, LED9.C
- net N$18: now also IC9.LED6, LED6.C; no longer IC7.P6, LED10.C
- net N$19: now also IC9.LED7, LED5.C; no longer IC7.P7, LED11.C
- net N$2: now also R9.1; no longer R6.1
- net N$20: now also LED5.A, R36.2; no longer LED11.A, R52.2
- net N$21: now also LED6.A, R37.2; no longer LED10.A, R51.2
- net N$22: now also LED7.A, R38.2; no longer LED9.A, R50.2
- net N$23: now also R39.2; no longer R49.2
- net N$24: now also LED9.A, R40.2; no longer LED7.A, R48.2
- net N$25: now also LED10.A, R41.2; no longer LED6.A, R47.2
- net N$26: now also LED11.A, R42.2; no longer LED5.A, R46.2
- net N$27: now also LED12.A, R43.2; no longer LED4.A, R45.2
- net N$28: now also LED4.A, R35.1; no longer LED12.A, R10.1
- net N$29: now also LED4.C, U5.D; no longer R11.2, T1.B
- net N$3: now also IC7.MODE, J4.2; no longer IC4.MODE, J2.2
- net N$30: now also R19.1, ST3.1; no longer LED12.C, T1.C
- net N$31: now also IC13.+OUT_L, J27.2; no longer C21.1, U6.BSN
- net N$32: now also IC13.-OUT_L, J27.1; no longer C22.1, U6.BSP
- net N$33: now also C25.1, IC13.VREF; no longer C23.1, U6.VCLAMP
- net N$35: now also IC4A.+IN, R21.2, R22.1; no longer C10.1, R14.S, R15.1
- net N$38: now also R4.1; no longer R1.1
- net N$39: now also IC5.!RST, U4.G; no longer C11.1, R20.S, R21.1
- net N$4: now also D1.A, D2.C, R1.2, R2.1, R3.2; no longer D3.AC, R7.2, R8.1, R9.2
- net N$45: now also R13.2, ST2.2; no longer R31.2, ST4.2
- net N$47: now also R12.1, ST1.2; no longer R30.1, ST3.2
- net N$5: now also IC4A.-IN, R24.1; no longer IC5A.-IN, R17.1
- net N$51: now also R14.1, ST1.5; no longer R32.1, ST3.5
- net N$53: now also R15.2, ST2.5; no longer R33.2, ST4.5
- net N$6: now also IC9.LED0, LED12.C; no longer IC7.P0, LED4.C
- net N$7: now also IC9.LED1, LED11.C; no longer IC7.P1, LED5.C
- net N$8: now also R7.2; no longer R4.2
- net N$9: now also C4.2, R5.1, R6.2; no longer C3.2, R2.1, R3.2
- net PWM_ERW_1: now also IC8.16/A2/PWM/T/ALT-SCL0, J22.1; no longer IC6.16/A2/PWM/T/ALT-SCL0, J21.1
- net PWM_ERW_2: now also IC8.17/A3/PWM/T/ALT-SDA0, J22.2; no longer IC6.17/A3/PWM/T/ALT-SDA0, J21.2
- net PWM_ERW_3: now also IC8.30/PWM/T/ALT-CAN0RX, J22.3, J6.9; no longer IC6.29/PWM/T/ALT-CAN0TX, J21.3
- net PWM_ERW_4: now also IC8.29/PWM/T/ALT-CAN0TX, J22.4; no longer IC6.30/PWM/T/ALT-CAN0RX, J21.4
- net PWM_ERW_5: now also IC8.4/PWM/SDA2/CAN0RX, J22.5; no longer IC6.3/PWM/SCL2/CAN0TX, J21.5
- net PWM_ERW_6: now also IC8.3/PWM/SCL2/CAN0TX, J22.6; no longer IC6.4/PWM/SDA2/CAN0RX, J21.6
- net RAD_L: now also C11.1, C12.1, IC4A.OUT, IC8.43/CS2-0, R22.2, R23.1; no longer C30.1, C31.1, IC5A.OUT, IC6.43/CS2-0, R16.2, R19.1
- net RAD_R: now also C14.1, C15.1, IC4B.OUT, IC8.44/MOSI2, R28.2, R29.1; no longer C28.1, C29.1, IC5B.OUT, IC6.44/MOSI2, R22.2, R25.1
- net RESET: now also IC8.RESET, J24.2, ST6.12, U4.D; no longer IC12./RST, IC6.RESET, J26.2, ST5.12
- net RX1: now also IC8.27/ALT-RX1/ALT-SCK0, ST6.15; no longer IC6.27/ALT-RX1/ALT-SCK0, J12.4, ST5.15
- net RX2: now also IC8.9/PWM/RX2/CS0-1, J15.4; no longer IC6.9/PWM/RX2/CS0-1, J8.4
- net RX5: now also IC8.34/A15/CAN1RX/RX5/ALT-SDA0, J16.4; no longer ESP-01.UTXD, IC6.34/A15/CAN1RX/RX5/ALT-SDA0
- net RX6: now also IC8.47/SCL0/RX6, J17.4; no longer IC6.47/SCL0/RX6, J13.4
- net SCL0: now also IC10.SCL, IC8.7/PWM/RX3/ALT-SCL0/ALT-MOSI0, IC9.SCL, J11.4, R45.1, ST6.21, U6.S; no longer IC6.7/PWM/RX3/ALT-SCL0/ALT-MOSI0, IC7.SCL, IC8.SCL, J10.4, R54.1, ST5.21, U4.S
- net SCL0_5V: now also J14.5, J5.4, R47.1, ST1.8, ST2.8, ST6.9, U6.D; no longer J7.5, J9.4, R56.1, ST5.9, U4.D
- net SCL1: now also IC8.37/A18/PWM/SCL1, J12.4; no longer IC6.37/A18/PWM/SCL1, J6.4
- net SCL3: now also IC8.57/SCL3/PWM, J13.3; no longer IC6.57/SCL3, J11.3
- net SDA0: now also IC10.SDA, IC8.8/PWM/TX3/ALT-SDA0/ALT-MISO0, IC9.SDA, J11.3, R44.1, ST6.19, U7.S; no longer IC6.8/PWM/TX3/ALT-SDA0/ALT-MISO0, IC7.SDA, IC8.SDA, J10.3, R53.1, ST5.19, U3.S
- net SDA0_5V: now also J14.4, J5.3, R46.1, ST1.7, ST2.7, ST6.7, U7.D; no longer J7.4, J9.3, R55.1, ST5.7, U3.D
- net SDA1: now also IC8.38/A19/PWM/SDA1, J12.3; no longer IC6.38/A19/PWM/SDA1, J6.3
- net SDA3: now also IC8.56/SDA3/PWM, J13.4; no longer IC6.56/SDA3, J11.4
- net SERVO1_FB: now also IC8.22/A8/PWM/T; no longer IC6.22/A8/PWM/T
- net SERVO1_PWM: now also IC8.5/PWM/ALT-TX1/ALT-MISO1, R34.1; no longer IC6.5/PWM/ALT-TX1/ALT-MISO1, R27.1
- net SERVO2_FB: now also IC8.23/A9/PWM/T, J19.4, ST6.20; no longer IC6.23/A9/PWM/T, J4.4, ST5.20
- net SERVO2_PWM: now also IC8.6/PWM, J19.3, R48.1, ST6.18; no longer IC6.6/PWM, J4.3, R28.1, ST5.18
- net SERVO3_PWM: now also IC8.25, J20.3, R49.1, ST6.16; no longer IC6.25, J5.3, R29.1
- net SERVO4_PWM: now also IC8.20/A6/PWM/CS0-2/ALT-SCK1, J21.1, J7.6; no longer IC6.20/A6/PWM/CS0-2/ALT-SCK1, J33.1
- net SERVO5_PWM: now also IC8.21/A7/PWM/CS0-3/ALT-MOSI1/ALT-RX1, J21.2, J7.7, J8.6; no longer IC6.21/A7/PWM/CS0-3/ALT-MOSI1/ALT-RX1, J33.2
- net SPI0_CS0: now also IC8.2/PWM, J6.6; no longer IC6.2/PWM, J16.3
- net SPI0_CS4: now also IC8.15/A1/CS0-4/T, J6.7; no longer IC6.15/A1/CS0-4/T, J16.4
- net SPI0_CS5: now also IC8.45/CS0-5/MISO2, J6.8; no longer IC6.45/CS0-5/MISO2, J16.5
- net SPI0_MISO: now also IC8.12/MISO0, J6.4, J7.4, J8.4; no longer IC6.12/MISO0, J16.7
- net SPI0_MOSI: now also IC8.11/MOSI0, J6.3, J7.3, J8.3; no longer IC6.11/MOSI0, J16.6
- net SPI0_SCK: now also IC8.14/A0/PWM/ALT-SCK0, J6.5, J7.5, J8.5; no longer IC6.14/A0/PWM/ALT-SCK0, J16.8
- net SPI1_CS0: now also IC8.31/A12/PWM/RX4/CS1-0, ST6.8; no longer IC6.31/A12/PWM/RX4/CS1-0, J17.3, ST5.8
- net SPI1_MISO: now also IC8.1/TX1/MISO1/T, ST6.2; no longer IC6.1/TX1/MISO1/T, J17.5, ST5.2
- net SPI1_MOSI: now also IC8.0/RX1/MOSI1/T, ST6.4; no longer IC6.0/RX1/MOSI1/T, J17.4, ST5.4
- net SPI1_SCK: now also IC8.32/A13/PWM/TX4/SCK1, ST6.6; no longer IC6.32/A13/PWM/TX4/SCK1, J17.6, ST5.6
- net SPI2_CS0: now also IC8.55, J9.6; no longer IC6.55, J18.3
- net SPI2_CS1: now also IC8.54/CS2-1, J10.6, J9.7; no longer IC6.54/CS2-1, J18.4
- net SPI2_MISO: now also IC8.51/MISO2, J10.4, J9.4; no longer IC6.51/MISO2, J18.6
- net SPI2_MOSI: now also IC8.52/MOSI2, J10.3, J9.3; no longer IC6.52/MOSI2, J18.5
- net SPI2_SCK: now also IC8.53/PWM/SCK2, J10.5, J9.5; no longer IC6.53/PWM/SCK2, J18.7
- net SWCLK: now also IC8.DC, J24.5; no longer IC6.DC, J26.5
- net SWDIO: now also IC8.DD, J24.6; no longer IC6.DD, J26.6
- net SWD_EN: now also IC8.DE, J24.4; no longer IC6.DE, J26.4
- net TX1: now also IC8.26/ALT-PWM/ALT-TX1/ALT-SCL2, ST6.17; no longer IC6.26/ALT-PWM/ALT-TX1/ALT-SCL2, J12.3, ST5.17
- net TX2: now also IC8.10/PWM/TX2/CS0-0, J15.3; no longer IC6.10/PWM/TX2/CS0-0, J8.3
- net TX5: now also IC8.33/A14/CAN1TX/TX5/ALT-SCL0, J16.3; no longer ESP-01.URXD, IC6.33/A14/CAN1TX/TX5/ALT-SCL0
- net TX6: now also IC8.48/SDA0/TX6, J17.3; no longer IC6.48/SDA0/TX6, J13.3
- net USB1_D+: now also IC8.D+, J133.3; no longer IC6.D+, J14.3
- net USB1_D-: now also IC8.D-, J133.2; no longer IC6.D-, J14.2
- net V5_L1: now also D4.C; no longer D2.C
- net V6_L1: now also D3.C; no longer D1.C
- net VBAT_RTC: now also IC8.VBAT; no longer IC6.VBAT
Other:
- note added: "(z.B. Display)"
- note added: "ESP12"
- note added: "Rev. 0.7"
- note added: "SERVO / PWM"
- note added: "TODO: SWD-Pins verbinden an GPIOs? Widerstaende?"
- note added: "ToDo: alternativ low-side switch (ULN 2803)?"
- note added: "ToDo: testen!"
- note added: "ToDo: testen! SHDN?"
- note added: "WIFI-Modul"
- note removed: "(Option A)"
- note removed: "(Option B)"
- note removed: "(o.ä. Reset-Controller)"
- note removed: "?"
- note removed: "Hinweis: Polung an Schraubklemme AK500-2-H vertauscht: jetzt identisch mit J25 Part in EAGLE Library con-ptr500 überführt"
- note removed: "RESET pruefen!"
- note removed: "RPI_SPI0_CE1 RPI_GPIO26 SERVO3_PWM RPI_3V3"
- note removed: "Rev. 0.6"
- note removed: "SERVO"
- note removed: "WIFI-Modul (optional)"
- moved on the sheet: BT1, C10, C11, C12, C14, C15, C21, C22, C23, C24, C25, C27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
