File: v2/boards/mcu_teensy.sch (EAGLE design)
At the start: 9 parts, among them Q1 BS108, U1 TEENSY3_6, U2 MCP101

Commit message: ct-Bot v2 prototype test boards updated/added
Simplified mainboard, teensy mcu board, and sensor boards are very early prototypes just for development and testing.
Other:
- note added: "Rev. 0.8.4"
- note removed: "Rev. 0.1.0"
Changed lines of the file:
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@@
 <?xml version="1.0" encoding="utf-8"?>
 <!DOCTYPE eagle SYSTEM "eagle.dtd">
-<eagle version="9.5.0">
+<eagle version="9.5.1">
 <drawing>
 <settings>
@@
 <text x="162.814" y="11.176" size="3.048" layer="94">c't-Bot v2 MCU Board
 !!! UNTESTED DRAFT !!!</text>
-<text x="217.17" y="20.32" size="2.54" layer="94">Rev. 0.1.0</text>
+<text x="217.17" y="20.32" size="2.54" layer="94">Rev. 0.8.4</text>
 <text x="162.814" y="5.842" size="2.54" layer="94">CC BY-SA 4.0</text>
 </plain>
@@
 <label x="121.92" y="53.34" size="1.778" layer="95"/>
 <pinref part="C1" gate="G$1" pin="1"/>
-<wire x1="119.38" y1="53.34" x2="114.3" y2="53.34" width="0.1524" layer="91"/>
 <wire x1="119.38" y1="50.8" x2="119.38" y2="53.34" width="0.1524" layer="91"/>
-<junction x="119.38" y="53.34"/>
-</segment>
-<segment>
+</segment>
+<segment>
