File: v2/boards/sensors_b.sch (EAGLE design)
At the start: 5 parts, among them U14 LINE_L, U15 LINE_R

Commit message: schematics and board files for ct-Bot v2 prototype
Parts:
- U14: value LINE_L -> LINE_R
- U15: value LINE_R -> LINE_L
Connections:
- net LINE_L: now also U15.COL; no longer U14.COL
- net LINE_R: now also U14.COL; no longer U15.COL
- net LOWSIDE_LINE_L: now also U15.C; no longer U14.C
- net LOWSIDE_LINE_R: now also U14.C; no longer U15.C
Other:
- note added: "Rev. 0.9.2"
- note added: "Timo Sandmann, CC BY-SA 4.0"
- note added: "ct-Bot v2 Liniensoren"
- note removed: "CC BY-SA 4.0"
- note removed: "Rev. 0.8.4"
- note removed: "c't-Bot v2 Liniensoren !!! UNTESTED DRAFT !!!"
Changed lines of the file:
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@@
 <?xml version="1.0" encoding="utf-8"?>
 <!DOCTYPE eagle SYSTEM "eagle.dtd">
-<eagle version="9.5.1">
+<eagle version="9.6.2">
 <drawing>
 <settings>
@@
 <parts>
 <part name="JP6" library="ct-bot" deviceset="PINHD-1X6" device=""/>
-<part name="U14" library="ct-bot" deviceset="CNY70" device="DEF" value="LINE_L"/>
-<part name="U15" library="ct-bot" deviceset="CNY70" device="DEF" value="LINE_R"/>
+<part name="U14" library="ct-bot" deviceset="CNY70" device="DEF" value="LINE_R"/>
+<part name="U15" library="ct-bot" deviceset="CNY70" device="DEF" value="LINE_L"/>
 <part name="FRAME1" library="frames" library_urn="urn:adsk.eagle:library:229" deviceset="DINA5_P" device=""/>
 <part name="SUPPLY1" library="supply2" library_urn="urn:adsk.eagle:library:372" deviceset="+5V" device=""/>
@@
 <sheet>
 <plain>
-<text x="33.274" y="11.176" size="3.048" layer="94">c't-Bot v2 Liniensoren
-!!! UNTESTED DRAFT !!!</text>
-<text x="87.63" y="20.32" size="2.54" layer="94">Rev. 0.8.4</text>
-<text x="33.274" y="5.842" size="2.54" layer="94">CC BY-SA 4.0</text>
-<text x="66.548" y="149.352" size="1.778" layer="97">Liniensensor L</text>
-<text x="66.548" y="118.872" size="1.778" layer="97">Liniensensor R</text>
+<text x="33.274" y="11.176" size="3.048" layer="94">ct-Bot v2 Liniensoren
+</text>
+<text x="87.63" y="20.32" size="2.54" layer="94">Rev. 0.9.2</text>
+<text x="33.274" y="5.842" size="2.54" layer="94">Timo Sandmann, CC BY-SA 4.0</text>
+<text x="66.548" y="149.352" size="1.778" layer="97">Liniensensor R</text>
+<text x="66.548" y="118.872" size="1.778" layer="97">Liniensensor L</text>
 </plain>
 <instances>
@@
 </busses>
 <nets>
+<net name="LOWSIDE_LINE_R" class="0">
+<segment>
+<pinref part="U14" gate="G$1" pin="C"/>
+<label x="20.32" y="157.48" size="1.778" layer="95"/>
+<pinref part="JP6" gate="A" pin="3"/>
+<wire x1="63.5" y1="157.48" x2="15.24" y2="157.48" width="0.1524" layer="91"/>
+</segment>
+</net>
 <net name="LOWSIDE_LINE_L" class="0">
 <segment>
-<pinref part="U14" gate="G$1" pin="C"/>
-<wire x1="63.5" y1="157.48" x2="60.96" y2="157.48" width="0.1524" layer="91"/>
-<wire x1="60.96" y1="157.48" x2="60.96" y2="160.02" width="0.1524" layer="91"/>
+<pinref part="U15" gate="G$1" pin="C"/>
+<wire x1="63.5" y1="127" x2="53.34" y2="127" width="0.1524" layer="91"/>
+<label x="20.32" y="160.02" size="1.778" layer="95"/>
+<wire x1="53.34" y1="127" x2="53.34" y2="160.02" width="0.1524" layer="91"/>
 <pinref part="JP6" gate="A" pin="2"/>
-<wire x1="60.96" y1="160.02" x2="15.24" y2="160.02" width="0.1524" layer="91"/>
-<label x="20.32" y="160.02" size="1.778" layer="95"/>
+<wire x1="53.34" y1="160.02" x2="15.24" y2="160.02" width="0.1524" layer="91"/>
 </segment>
 </net>
-<net name="LOWSIDE_LINE_R" class="0">
-<segment>
-<pinref part="U15" gate="G$1" pin="C"/>
-<wire x1="63.5" y1="127" x2="55.88" y2="127" width="0.1524" layer="91"/>
-<wire x1="55.88" y1="127" x2="55.88" y2="157.48" width="0.1524" layer="91"/>
-<pinref part="JP6" gate="A" pin="3"/>
-<wire x1="55.88" y1="157.48" x2="15.24" y2="157.48" width="0.1524" layer="91"/>
-<label x="20.32" y="157.48" size="1.778" layer="95"/>
-</segment>
-</net>
-<net name="LINE_L" class="0">
+<net name="LINE_R" class="0">
 <segment>
 <pinref part="U14" gate="G$1" pin="COL"/>
 <wire x1="81.28" y1="162.56" x2="83.82" y2="162.56" width="0.1524" layer="91"/>
 <wire x1="83.82" y1="162.56" x2="83.82" y2="147.32" width="0.1524" layer="91"/>
-<wire x1="83.82" y1="147.32" x2="53.34" y2="147.32" width="0.1524" layer="91"/>
-<wire x1="53.34" y1="147.32" x2="53.34" y2="154.94" width="0.1524" layer="91"/>
-<pinref part="JP6" gate="A" pin="4"/>
-<wire x1="53.34" y1="154.94" x2="15.24" y2="154.94" width="0.1524" layer="91"/>
-<label x="20.32" y="154.94" size="1.778" layer="95"/>
+<wire x1="83.82" y1="147.32" x2="48.26" y2="147.32" width="0.1524" layer="91"/>
+<label x="20.32" y="152.4" size="1.778" layer="95"/>
+<pinref part="JP6" gate="A" pin="5"/>
+<wire x1="48.26" y1="147.32" x2="48.26" y2="152.4" width="0.1524" layer="91"/>
+<wire x1="48.26" y1="152.4" x2="15.24" y2="152.4" width="0.1524" layer="91"/>
 </segment>
 </net>
-<net name="LINE_R" class="0">
+<net name="LINE_L" class="0">
 <segment>
 <pinref part="U15" gate="G$1" pin="COL"/>
@@
 <wire x1="83.82" y1="132.08" x2="83.82" y2="144.78" width="0.1524" layer="91"/>
 <wire x1="83.82" y1="144.78" x2="50.8" y2="144.78" width="0.1524" layer="91"/>
-<pinref part="JP6" gate="A" pin="5"/>
-<wire x1="50.8" y1="144.78" x2="50.8" y2="152.4" width="0.1524" layer="91"/>
-<wire x1="50.8" y1="152.4" x2="15.24" y2="152.4" width="0.1524" layer="91"/>
-<label x="20.32" y="152.4" size="1.778" layer="95"/>
+<label x="20.32" y="154.94" size="1.778" layer="95"/>
+<wire x1="50.8" y1="144.78" x2="50.8" y2="154.94" width="0.1524" layer="91"/>
+<pinref part="JP6" gate="A" pin="4"/>
+<wire x1="50.8" y1="154.94" x2="15.24" y2="154.94" width="0.1524" layer="91"/>
 </segment>
 </net>
